File: hardware/kicad/tuner.kicad_pcb (KiCad board)
At the start: 4 copper layers, 100 x 70 mm, 61 parts, among them J1 12V_IN, J2 RADIO_UNIVERSAL, J3 RF_IN_SO239, J4 RF_OUT_SO239, J5 EXT_SWR, J6 ANT_CTRL, J8 DEBUG_UART, Q1 MMBT3904, Q2 MMBT3904, SW1 TUNE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

Commit message: Revise power stage and refresh hardware artifacts
Parts:
- removed J5: EXT_SWR, Jack_3.5mm_CUI_SJ1-3533NG_Horizontal
- U1: value MP1584_3V3 -> OKI78SR_3V3; footprint BUCK_MP1584 -> REG_OKI78SR
- moved U1 10.8 mm to (156.5, 88.0)
- moved C3 10.0 mm to (166.5, 92.0), turned to 90 degrees
- moved C2 6.32 mm to (155.5, 96.0)
- moved C_VM 6.32 mm to (159.5, 104.0)
- moved C7 4.00 mm to (165.5, 116.0)
- moved C1 3.00 mm to (140.5, 94.0)
- moved D1 3.00 mm to (147.5, 84.0)
- moved F1 3.00 mm to (139.5, 84.0)
